Commit message: WIP: to squash

File: third_party_examples/drake_examples/panda/robots/panda_arm.urdf (robot description, URDF)
Before this commit: robot panda, 9 links, 8 joints
Links:
- added link base
- link panda_link0: mass None -> 5
- link panda_link1: mass None -> 4.970684
- link panda_link2: mass None -> 0.646926
- link panda_link3: mass None -> 3.228604
- link panda_link4: mass None -> 3.587895
- link panda_link5: mass None -> 1.225946
- link panda_link6: mass None -> 1.666555
- link panda_link7: mass None -> 7.35522e-01
- link panda_link8: mass None -> 0.0
Joints:
- added joint panda_base_joint: type fixed, parent base, child panda_link0, origin xyz=0 0 0 rpy=0 0 0

Commit message: fix(drake): Use the stable version

File: third_party_examples/drake_examples/panda/robots/panda_arm.urdf (robot description, URDF)
Before this commit: robot panda, 10 links, 9 joints
Links:
- removed link base
- link panda_link0: mass 5 -> 2.92; geometry collision sphere radius=0.06; collision sphere radius=0.06
- link panda_link1: mass 4.970684 -> 2.74; geometry collision sphere radius=0.06; collision sphere radius=0.06
- link panda_link2: mass 0.646926 -> 2.74; geometry collision sphere radius=0.06; collision sphere radius=0.06
- link panda_link3: mass 3.228604 -> 2.38; geometry collision sphere radius=0.06; collision sphere radius=0.06
- link panda_link4: mass 3.587895 -> 2.38; geometry collision sphere radius=0.05; collision sphere radius=0.055
- link panda_link5: mass 1.225946 -> 2.74; geometry collision sphere radius=0.035; collision sphere radius=0.035
- link panda_link6: mass 1.666555 -> 1.55; geometry collision sphere radius=0.05; collision sphere radius=0.06
- link panda_link7: mass 7.35522e-01 -> 0.54; geometry collision sphere radius=0.05; collision sphere radius=0.06
- link panda_link8: mass 0.0 -> None; geometry collision sphere radius=0.04
Joints:
- removed joint panda_base_joint
- joint panda_joint2: origin xyz=0 0 0 rpy=-1.5707963267948966 0 0 -> xyz=0 0 0 rpy=-1.57079632679 0 0
- joint panda_joint3: origin xyz=0 -0.316 0 rpy=1.5707963267948966 0 0 -> xyz=0 -0.316 0 rpy=1.57079632679 0 0
- joint panda_joint4: origin xyz=0.0825 0 0 rpy=1.5707963267948966 0 0 -> xyz=0.0825 0 0 rpy=1.57079632679 0 0
- joint panda_joint5: limit lower=-2.8973 upper=2.8973 effort=12 velocity=2.6100 -> lower=-2.8973 upper=2.8973 effort=12 velocity=2.610; origin xyz=-0.0825 0.384 0 rpy=-1.5707963267948966 0 0 -> xyz=-0.0825 0.384 0 rpy=-1.57079632679 0 0
- joint panda_joint6: limit lower=-0.0175 upper=3.7525 effort=12 velocity=2.6100 -> lower=-0.0175 upper=3.7525 effort=12 velocity=2.610; origin xyz=0 0 0 rpy=1.5707963267948966 0 0 -> xyz=0 0 0 rpy=1.57079632679 0 0
- joint panda_joint7: limit lower=-2.8973 upper=2.8973 effort=12 velocity=2.6100 -> lower=-2.8973 upper=2.8973 effort=12 velocity=2.610; origin xyz=0.088 0 0 rpy=1.5707963267948966 0 0 -> xyz=0.088 0 0 rpy=1.57079632679 0 0
